File: Jason's PCB.sch (KiCad schematic (older format))
At the start: 11 parts, among them U1 Elite-C

Commit message: Formatting
-Changes some labels
Parts:
- SW_E1, SW_E2: footprint (none) -> Keebio-Parts:RotaryEncoder_EC11
Changed lines of the file:
@@
 F 0 "SW_E1" H 5550 2667 50  0000 C CNN
 F 1 "Rotary_Encoder_Switch" H 5550 2576 50  0000 C CNN
-F 2 "" H 5400 2460 50  0001 C CNN
+F 2 "Keebio-Parts:RotaryEncoder_EC11" H 5400 2460 50  0001 C CNN
 F 3 "~" H 5550 2560 50  0001 C CNN
 	1    5550 2300
@@
 F 0 "SW_E2" H 5550 3317 50  0000 C CNN
 F 1 "Rotary_Encoder_Switch" H 5550 3226 50  0000 C CNN
-F 2 "" H 5400 3110 50  0001 C CNN
+F 2 "Keebio-Parts:RotaryEncoder_EC11" H 5400 3110 50  0001 C CNN
 F 3 "~" H 5550 3210 50  0001 C CNN
 	1    5550 2950
@@
 SWD3
 $Comp
-L power:GND #PWR?
+L power:GND #PWR0107
 U 1 1 5E053B0E
 P 5850 2200
-F 0 "#PWR?" H 5850 1950 50  0001 C CNN
+F 0 "#PWR0107" H 5850 1950 50  0001 C CNN
 F 1 "GND" V 5855 2072 50  0000 R CNN
 F 2 "" H 5850 2200 50  0001 C CNN
@@
 $EndComp
 $Comp
-L power:GND #PWR?
+L power:GND #PWR0108
 U 1 1 5E0546A3
 P 5850 2850
-F 0 "#PWR?" H 5850 2600 50  0001 C CNN
+F 0 "#PWR0108" H 5850 2600 50  0001 C CNN
 F 1 "GND" V 5855 2722 50  0000 R CNN
 F 2 "" H 5850 2850 50  0001 C CNN
@@
 $EndComp
 $Comp
-L power:GND #PWR?
+L power:GND #PWR0109
 U 1 1 5E0555B2
 P 5250 2300
-F 0 "#PWR?" H 5250 2050 50  0001 C CNN
+F 0 "#PWR0109" H 5250 2050 50  0001 C CNN
 F 1 "GND" V 5255 2172 50  0000 R CNN
 F 2 "" H 5250 2300 50  0001 C CNN
@@
 $EndComp
 $Comp
-L power:GND #PWR?
+L power:GND #PWR0110
 U 1 1 5E05630C
 P 5250 2950
-F 0 "#PWR?" H 5250 2700 50  0001 C CNN
+F 0 "#PWR0110" H 5250 2700 50  0001 C CNN
 F 1 "GND" V 5255 2822 50  0000 R CNN
 F 2 "" H 5250 2950 50  0001 C CNN
